Commit message: the working model with proper URDF without Aruco. view_urdf.launch is for loading urdf onto param server and gazebo.launch is for spwaning bot in gazebo world. At present two bots have been launched and the code can be scaled for more

File: software/bot_description/urdf/bot.urdf (robot description, URDF)
Before this commit: robot bot, 1 links, 0 joints
Links:
- added link base_link_inertia, mass 1; collision box size=0.12 0.12 0.008; visual box size=0.12 0.12 0.008
- added link caster_wheel, mass 3; collision sphere radius=0.0283333333333; visual sphere radius=0.0283333333333
- added link left_wheel, mass 0.3; collision cylinder length=0.008 radius=0.0425; visual cylinder length=0.008 radius=0.0425
- added link right_wheel, mass 0.3; collision cylinder length=0.008 radius=0.0425; visual cylinder length=0.008 radius=0.0425
- link base_link: geometry 
Joints:
- added joint base_link_inertia_joint: type fixed, parent base_link, child base_link_inertia, origin xyz=0 0 0 rpy=0 0 0
- added joint caster_wheel_joint: type continuous, parent base_link, child caster_wheel, origin xyz=0.04 0 -0.0491666666667 rpy=0 0 0, axis 0 1 0
- added joint left_wheel_joint: type continuous, parent base_link, child left_wheel, origin xyz=-0.04 0.068  -0.035 rpy=0 1.570795 1.570795, axis 0 0 1
- added joint right_wheel_joint: type continuous, parent base_link, child right_wheel, origin xyz=-0.04 -0.068  -0.035 rpy=0 1.570795 1.570795, axis 0 0 1

File: software/bot_description/urdf/bot.urdf.xacro (robot description, xacro)
@@ -6,7 +6,17 @@
 	<xacro:property name="length" value="0.12"/>
 	<xacro:property name="breadth" value="0.12"/>
-	<link name="base_link">
+	<xacro:property name="pi" value="3.14159"/>
+	<xacro:property name="m_base" value="1"/>
+	<xacro:property name="m_wheel" value="0.3"/>
+	<xacro:property name="m_caster_wheel" value="3"/>
+	<link name="base_link"/>
+	<link name="base_link_inertia">
+		<inertial>
+     		<origin xyz="0 0 0" rpy="0 0 0"/>
+     		<mass value="${m_base}"/>
+     		<inertia ixx="${m_base*(breadth*breadth+0.008*0.008)/12.0}"  ixy="0"  ixz="0" iyy="${m_base*(length*length+0.008*0.008)/12.0}" iyz="0" izz="${m_base*(breadth*breadth+length*length)/12.0}" />
+   		</inertial>
 		<collision>
-			<origin xyz="0 0 ${bot_height}" rpy="0 0 0"/>
+			<origin xyz="0 0 0" rpy="0 0 0"/>
 			<geometry>
 				<box size="${length} ${breadth} 0.008"/>
@@ -14,5 +24,5 @@
 		</collision>
 		<visual>
-			<origin xyz="0 0 ${bot_height}" rpy="0 0 0"/>
+			<origin xyz="0 0 0" rpy="0 0 0"/>
 			<geometry>
 				<box size="${length} ${breadth} 0.008"/>
@@ -21,17 +31,97 @@
 	</link>
 	<link name="left_wheel">
+		<inertial>
+     		<origin xyz="0 0 0" rpy="0 0 0"/>
+     		<mass value="${m_wheel}"/>
+     		<inertia ixx="${m_wheel*(3*wheel_dia*wheel_dia/4.0+0.008*0.008)/12.0}"  ixy="0"  ixz="0" iyy="${m_wheel*(3*wheel_dia*wheel_dia/4.0+0.008*0.008)/12.0}" iyz="0" izz="${m_wheel*(wheel_dia*wheel_dia/4)/2.0}" />
+   		</inertial>
 		<collision>
 			<origin xyz="0 0 0" rpy="0 0 0"/>
 			<geometry>
-				<cylinder radius="${wheel_dia/2}" length="0.008"/>
+				<cylinder radius="${wheel_dia/2.0}" length="0.008"/>
 			</geometry>
 		</collision>
 		<visual>
-			<origin xyz="${length/2} -0.4 -0.35" rpy="0 0 0"/>
+			<origin xyz="0 0 0" rpy="0 0 0"/>
 			<geometry>
-				<cylinder radius="${wheel_dia/2}" length="0.008"/>
+				<cylinder radius="${wheel_dia/2.0}" length="0.008"/>
 			</geometry>
 		</visual>
 	</link>
-	${length/2} -0.4 -0.35
+	<link name="right_wheel">
+		<inertial>
+     		<origin xyz="0 0 0" rpy="0 0 0"/>
+     		<mass value="${m_wheel}"/>
+     		<inertia ixx="${m_wheel*(3*wheel_dia*wheel_dia/4.0+0.008*0.008)/12.0}"  ixy="0"  ixz="0" iyy="${m_wheel*(3*wheel_dia*wheel_dia/4.0+0.008*0.008)/12.0}" iyz="0" izz="${m_wheel*(wheel_dia*wheel_dia/4)/2.0}" />
+   		</inertial>
+		<collision>
+			<origin xyz="0 0 0" rpy="0 0 0"/>
+			<geometry>
+				<cylinder radius="${wheel_dia/2.0}" length="0.008"/>
+			</geometry>
+		</collision>
+		<visual>
+			<origin xyz="0 0 0" rpy="0 0 0"/>
+			<geometry>
+				<cylinder radius="${wheel_dia/2.0}" length="0.008"/>
+			</geometry>
+		</visual>
+	</link>
+	<link name="caster_wheel">
+		<inertial>
+     		<origin xyz="0 0 0" rpy="0 0 0"/>
+     		<mass value="${m_caster_wheel}"/>
+     		<inertia ixx="${m_caster_wheel*(2*wheel_dia*wheel_dia/9.0)/5.0}"  ixy="0"  ixz="0" iyy="${m_caster_wheel*(2*wheel_dia*wheel_dia/9.0)/5.0}" iyz="0" izz="${m_caster_wheel*(2*wheel_dia*wheel_dia/9.0)/5.0}" />
+   		</inertial>
+		<collision>
+			<origin xyz="0 0 0" rpy="0 0 0"/>
+			<geometry>
+				<sphere radius="${wheel_dia/3.0}"/>
+			</geometry>
+		</collision>
+		<visual>
+			<origin xyz="0 0 0" rpy="0 0 0"/>
+			<geometry>
+				<sphere radius="${wheel_dia/3.0}"/>
+			</geometry>
+		</visual>
+	</link>
+	<joint name="base_link_inertia_joint" type="fixed">
+		<parent link="base_link"/>
+		<child link="base_link_inertia"/>
+		<origin rpy="0 0 0" xyz="0 0 0"/>
+	</joint>
+	<joint name="left_wheel_joint" type="continuous">
+		<parent link="base_link"/>
+		<child link="left_wheel"/>
+		<origin rpy="0 ${pi/2} ${pi/2}" xyz="-0.04 ${breadth/2+0.008}  -0.035"/>
+		<axis rpy="0 0 0" xyz="0 0 1"/>
+	</joint>
+	<joint name="right_wheel_joint" type="continuous">
+		<parent link="base_link"/>
+		<child link="right_wheel"/>
+		<origin rpy="0 ${pi/2} ${pi/2}" xyz="-0.04 ${-breadth/2-0.008}  -0.035"/>
+		<axis rpy="0 0 0" xyz="0 0 1"/>
+	</joint>
+	<joint name="caster_wheel_joint" type="continuous">
+		<parent link="base_link"/>
+		<child link="caster_wheel"/>
+		<origin rpy="0 0 0" xyz="${length/2-0.02} 0 ${-0.035- wheel_dia/6}"/>
+		<axis rpy="0 0 0" xyz="0 1 0"/>
+	</joint>
+	<gazebo>
+    <plugin filename="libgazebo_ros_diff_drive.so" name="differential_drive_controller">
+      <alwaysOn>true</alwaysOn>
+      <updateRate>20</updateRate>
+      <leftJoint>left_wheel_joint</leftJoint>
+      <rightJoint>right_wheel_joint</rightJoint>
+      <wheelSeparation>${breadth+0.016}</wheelSeparation>
+      <wheelDiameter>${wheel_dia}</wheelDiameter>
+      <torque>0.1</torque>
+      <commandTopic>cmd_vel</commandTopic>
+      <odometryTopic>odom</odometryTopic>
+      <odometryFrame>odom</odometryFrame>
+      <robotBaseFrame>base_link</robotBaseFrame>
+    </plugin>
+  </gazebo>
 </robot>

Commit message: cerated 4 diff urdf of bot with diff aruco. meshes of base with arcuo can be found in bot_description/meshes. Need to get the arena_world setup for which image has been mae and also texture. but it couldnt be insterted into world yet

File: software/bot_description/urdf/bot.urdf (robot description, URDF)
Before this commit: robot bot, 5 links, 4 joints
Links:
- link base_link_inertia: geometry collision box size=0.12 0.12 0.008; visual mesh filename=package://bot_description/meshes/bot1.dae

File: software/bot_description/urdf/bot.urdf.xacro (robot description, xacro)
@@ -26,5 +26,5 @@
 			<origin xyz="0 0 0" rpy="0 0 0"/>
 			<geometry>
-				<box size="${length} ${breadth} 0.008"/>
+				<mesh filename="package://bot_description/meshes/bot4.dae"  />
 			</geometry>
 		</visual>
