Commit message: final working urdf with arena 4 bots and camera plugin. Now the bots move a bot only that thing needs to be resolved

File: software/bot_description/urdf/arena.urdf (robot description, URDF)
Before this commit: robot bot, 2 links, 1 joints
Links:
- added link camera_link, mass 1e-5; collision box size=0.05 0.05 0.05; visual box size=0.05 0.05 0.05
- link arena: mass None -> 1; geometry collision box size=0.0001 0.0001 0.0001; visual mesh filename=package://bot_description/meshes/arena1.dae
Joints:
- added joint camera_joint: type fixed, parent world, child camera_link, origin xyz=0 0 1.8 rpy=0 1.517 0, axis 0 1 0
- joint world_arena: origin xyz=0 0 0 rpy=0 0 0 -> xyz=0 0 0.0001 rpy=0 0 0

File: software/bot_description/urdf/bot.urdf.xacro (robot description, xacro)
@@ -2,8 +2,8 @@
 <robot name="bot" xmlns:xacro="http://ros.org/wiki/xacro">
 	<!-- <xacro:include filename="$(find bot_description)/urdf/" /> -->
-	<xacro:property name="wheel_dia" value="0.085"/>
-	<xacro:property name="bot_height" value="0.115"/>
-	<xacro:property name="length" value="0.12"/>
-	<xacro:property name="breadth" value="0.12"/>
+	<xacro:property name="wheel_dia" value="0.05"/>
+	<xacro:property name="bot_height" value="0.07"/>
+	<xacro:property name="length" value="0.08"/>
+	<xacro:property name="breadth" value="0.08"/>
 	<xacro:property name="pi" value="3.14159"/>
 	<xacro:property name="m_base" value="1"/>
@@ -26,5 +26,5 @@
 			<origin xyz="0 0 0" rpy="0 0 0"/>
 			<geometry>
-				<mesh filename="package://bot_description/meshes/bot4.dae"  />
+				<mesh filename="package://bot_description/meshes/bot1.dae"  />
 			</geometry>
 		</visual>
@@ -95,5 +95,5 @@
 		<parent link="base_link"/>
 		<child link="left_wheel"/>
-		<origin rpy="0 ${pi/2} ${pi/2}" xyz="-0.04 ${breadth/2+0.008}  -0.035"/>
+		<origin rpy="0 ${pi/2} ${pi/2}" xyz="-0.02 ${breadth/2+0.008}  -0.015"/>
 		<axis rpy="0 0 0" xyz="0 0 1"/>
 	</joint>
@@ -101,5 +101,5 @@
 		<parent link="base_link"/>
 		<child link="right_wheel"/>
-		<origin rpy="0 ${pi/2} ${pi/2}" xyz="-0.04 ${-breadth/2-0.008}  -0.035"/>
+		<origin rpy="0 ${pi/2} ${pi/2}" xyz="-0.02 ${-breadth/2-0.008}  -0.015"/>
 		<axis rpy="0 0 0" xyz="0 0 1"/>
 	</joint>
@@ -107,5 +107,5 @@
 		<parent link="base_link"/>
 		<child link="caster_wheel"/>
-		<origin rpy="0 0 0" xyz="${length/2-0.02} 0 ${-0.035- wheel_dia/6}"/>
+		<origin rpy="0 0 0" xyz="${length/2-0.02} 0 ${-0.015- wheel_dia/6}"/>
 		<axis rpy="0 0 0" xyz="0 1 0"/>
 	</joint>
@@ -118,5 +118,5 @@
       <wheelSeparation>${breadth+0.016}</wheelSeparation>
       <wheelDiameter>${wheel_dia}</wheelDiameter>
-      <torque>0.1</torque>
+      <torque>0.001</torque>
       <commandTopic>cmd_vel</commandTopic>
       <odometryTopic>odom</odometryTopic>

File: software/bot_description/urdf/bot1.urdf (robot description, URDF)
Before this commit: robot bot, 5 links, 4 joints
Links:
- link base_link_inertia: geometry collision box size=0.08 0.08 0.008; visual mesh filename=package://bot_description/meshes/bot1.dae
- link caster_wheel: geometry collision sphere radius=0.0166666666667; visual sphere radius=0.0166666666667
- link left_wheel: geometry collision cylinder length=0.008 radius=0.025; visual cylinder length=0.008 radius=0.025
- link right_wheel: geometry collision cylinder length=0.008 radius=0.025; visual cylinder length=0.008 radius=0.025
Joints:
- joint caster_wheel_joint: origin xyz=0.04 0 -0.0491666666667 rpy=0 0 0 -> xyz=0.02 0 -0.0233333333333 rpy=0 0 0
- joint left_wheel_joint: origin xyz=-0.04 0.068  -0.035 rpy=0 1.570795 1.570795 -> xyz=-0.02 0.048  -0.015 rpy=0 1.570795 1.570795
- joint right_wheel_joint: origin xyz=-0.04 -0.068  -0.035 rpy=0 1.570795 1.570795 -> xyz=-0.02 -0.048  -0.015 rpy=0 1.570795 1.570795

File: software/bot_description/urdf/bot2.urdf (robot description, URDF)
Before this commit: robot bot, 5 links, 4 joints
Links:
- link base_link_inertia: geometry collision box size=0.08 0.08 0.008; visual mesh filename=package://bot_description/meshes/bot2.dae
- link caster_wheel: geometry collision sphere radius=0.0166666666667; visual sphere radius=0.0166666666667
- link left_wheel: geometry collision cylinder length=0.008 radius=0.025; visual cylinder length=0.008 radius=0.025
- link right_wheel: geometry collision cylinder length=0.008 radius=0.025; visual cylinder length=0.008 radius=0.025
Joints:
- joint caster_wheel_joint: origin xyz=0.04 0 -0.0491666666667 rpy=0 0 0 -> xyz=0.02 0 -0.0233333333333 rpy=0 0 0
- joint left_wheel_joint: origin xyz=-0.04 0.068  -0.035 rpy=0 1.570795 1.570795 -> xyz=-0.02 0.048  -0.015 rpy=0 1.570795 1.570795
- joint right_wheel_joint: origin xyz=-0.04 -0.068  -0.035 rpy=0 1.570795 1.570795 -> xyz=-0.02 -0.048  -0.015 rpy=0 1.570795 1.570795

File: software/bot_description/urdf/bot3.urdf (robot description, URDF)
Before this commit: robot bot, 5 links, 4 joints
Links:
- link base_link_inertia: geometry collision box size=0.08 0.08 0.008; visual mesh filename=package://bot_description/meshes/bot3.dae
- link caster_wheel: geometry collision sphere radius=0.0166666666667; visual sphere radius=0.0166666666667
- link left_wheel: geometry collision cylinder length=0.008 radius=0.025; visual cylinder length=0.008 radius=0.025
- link right_wheel: geometry collision cylinder length=0.008 radius=0.025; visual cylinder length=0.008 radius=0.025
Joints:
- joint caster_wheel_joint: origin xyz=0.04 0 -0.0491666666667 rpy=0 0 0 -> xyz=0.02 0 -0.0233333333333 rpy=0 0 0
- joint left_wheel_joint: origin xyz=-0.04 0.068  -0.035 rpy=0 1.570795 1.570795 -> xyz=-0.02 0.048  -0.015 rpy=0 1.570795 1.570795
- joint right_wheel_joint: origin xyz=-0.04 -0.068  -0.035 rpy=0 1.570795 1.570795 -> xyz=-0.02 -0.048  -0.015 rpy=0 1.570795 1.570795

File: software/bot_description/urdf/bot4.urdf (robot description, URDF)
Before this commit: robot bot, 5 links, 4 joints
Links:
- link base_link_inertia: geometry collision box size=0.08 0.08 0.008; visual mesh filename=package://bot_description/meshes/bot4.dae
- link caster_wheel: geometry collision sphere radius=0.0166666666667; visual sphere radius=0.0166666666667
- link left_wheel: geometry collision cylinder length=0.008 radius=0.025; visual cylinder length=0.008 radius=0.025
- link right_wheel: geometry collision cylinder length=0.008 radius=0.025; visual cylinder length=0.008 radius=0.025
Joints:
- joint caster_wheel_joint: origin xyz=0.04 0 -0.0491666666667 rpy=0 0 0 -> xyz=0.02 0 -0.0233333333333 rpy=0 0 0
- joint left_wheel_joint: origin xyz=-0.04 0.068  -0.035 rpy=0 1.570795 1.570795 -> xyz=-0.02 0.048  -0.015 rpy=0 1.570795 1.570795
- joint right_wheel_joint: origin xyz=-0.04 -0.068  -0.035 rpy=0 1.570795 1.570795 -> xyz=-0.02 -0.048  -0.015 rpy=0 1.570795 1.570795

Commit message: aruco detection has been implemented though it needs to be fine tuned a bit for reliability

File: software/bot_description/urdf/arena.urdf (robot description, URDF)
Before this commit: robot arena1, 3 links, 2 joints
Joints:
- joint camera_joint: origin xyz=0 0 1.8 rpy=0 1.517 0 -> xyz=0 0 1.2 rpy=0 1.517 0

File: software/bot_description/urdf/bot1.urdf (robot description, URDF)
Before this commit: robot bot1, 5 links, 4 joints
Joints:
- joint left_wheel_joint: origin xyz=-0.02 0.048  -0.015 rpy=0 1.570795 1.570795 -> xyz=-0.02 0.058  -0.015 rpy=0 1.570795 1.570795
- joint right_wheel_joint: origin xyz=-0.02 -0.048  -0.015 rpy=0 1.570795 1.570795 -> xyz=-0.02 -0.058  -0.015 rpy=0 1.570795 1.570795

File: software/bot_description/urdf/bot2.urdf (robot description, URDF)
Before this commit: robot bot2, 5 links, 4 joints
Joints:
- joint left_wheel_joint: origin xyz=-0.02 0.048  -0.015 rpy=0 1.570795 1.570795 -> xyz=-0.02 0.058  -0.015 rpy=0 1.570795 1.570795
- joint right_wheel_joint: origin xyz=-0.02 -0.048  -0.015 rpy=0 1.570795 1.570795 -> xyz=-0.02 -0.058  -0.015 rpy=0 1.570795 1.570795

File: software/bot_description/urdf/bot3.urdf (robot description, URDF)
Before this commit: robot bot3, 5 links, 4 joints
Joints:
- joint left_wheel_joint: origin xyz=-0.02 0.048  -0.015 rpy=0 1.570795 1.570795 -> xyz=-0.02 0.058  -0.015 rpy=0 1.570795 1.570795
- joint right_wheel_joint: origin xyz=-0.02 -0.048  -0.015 rpy=0 1.570795 1.570795 -> xyz=-0.02 -0.058  -0.015 rpy=0 1.570795 1.570795

File: software/bot_description/urdf/bot4.urdf (robot description, URDF)
Before this commit: robot bot4, 5 links, 4 joints
Joints:
- joint left_wheel_joint: origin xyz=-0.02 0.048  -0.015 rpy=0 1.570795 1.570795 -> xyz=-0.02 0.058  -0.015 rpy=0 1.570795 1.570795
- joint right_wheel_joint: origin xyz=-0.02 -0.048  -0.015 rpy=0 1.570795 1.570795 -> xyz=-0.02 -0.058  -0.015 rpy=0 1.570795 1.570795

Commit message: aruco detection completed

File: software/bot_description/urdf/arena.urdf (robot description, URDF)
Before this commit: robot arena1, 3 links, 2 joints
Joints:
- joint camera_joint: origin xyz=0 0 1.2 rpy=0 1.517 0 -> xyz=0 0 1.2 rpy=0 1.57079632679 0

Commit message: .

File: software/bot_description/urdf/arena.urdf (robot description, URDF)
Before this commit: robot arena1, 3 links, 2 joints
Joints:
- joint camera_joint: origin xyz=0 0 1.2 rpy=0 1.57079632679 0 -> xyz=0 0 1.4 rpy=0 1.57079632679 0

File: software/bot_description/urdf/bot.urdf.xacro (robot description, xacro)
@@ -1,4 +1,4 @@
 <?xml version="1.0"?>
-<robot name="bot1" xmlns:xacro="http://ros.org/wiki/xacro">
+<robot name="bot4" xmlns:xacro="http://ros.org/wiki/xacro">
 	<xacro:property name="wheel_dia" value="0.05"/>
 	<xacro:property name="bot_height" value="0.07"/>
@@ -9,5 +9,5 @@
 	<xacro:property name="m_wheel" value="0.3"/>
 	<xacro:property name="m_caster_wheel" value="3"/>
-  <xacro:property name="bot_number" value="1"/>
+  <xacro:property name="bot_number" value="4"/>
 	<link name="base_link"/>
 	<link name="base_link_inertia">
@@ -24,7 +24,7 @@
 		</collision>
 		<visual>
-			<origin xyz="0 0 0" rpy="0 0 0"/>
+			<origin xyz="0 0 0.02" rpy="0 0 0"/>
 			<geometry>
-				<mesh filename="package://bot_description/meshes/bot${bot_number}.dae"  />
+				<mesh filename="package://bot_description/meshes/bot${bot_number}.dae" scale="1.22 1.22 1.22"  />
 			</geometry>
 		</visual>

File: software/bot_description/urdf/bot1.urdf (robot description, URDF)
Before this commit: robot bot1, 5 links, 4 joints
Links:
- link base_link_inertia: geometry collision box size=0.08 0.08 0.008; visual mesh filename=package://bot_description/meshes/bot1.dae scale=1.22 1.22 1.22
Joints:
- removed joint left_wheel_joint
- removed joint right_wheel_joint
- added joint bot1_left_wheel_joint: type continuous, parent base_link, child left_wheel, origin xyz=-0.02 0.048  -0.015 rpy=0 1.570795 1.570795, axis 0 0 1
- added joint bot1_right_wheel_joint: type continuous, parent base_link, child right_wheel, origin xyz=-0.02 -0.048  -0.015 rpy=0 1.570795 1.570795, axis 0 0 1

File: software/bot_description/urdf/bot2.urdf (robot description, URDF)
Before this commit: robot bot2, 5 links, 4 joints
Links:
- link base_link_inertia: geometry collision box size=0.08 0.08 0.008; visual mesh filename=package://bot_description/meshes/bot2.dae scale=1.22 1.22 1.22
Joints:
- removed joint left_wheel_joint
- removed joint right_wheel_joint
- added joint bot2_left_wheel_joint: type continuous, parent base_link, child left_wheel, origin xyz=-0.02 0.048  -0.015 rpy=0 1.570795 1.570795, axis 0 0 1
- added joint bot2_right_wheel_joint: type continuous, parent base_link, child right_wheel, origin xyz=-0.02 -0.048  -0.015 rpy=0 1.570795 1.570795, axis 0 0 1

File: software/bot_description/urdf/bot3.urdf (robot description, URDF)
Before this commit: robot bot3, 5 links, 4 joints
Links:
- link base_link_inertia: geometry collision box size=0.08 0.08 0.008; visual mesh filename=package://bot_description/meshes/bot3.dae scale=1.22 1.22 1.22
Joints:
- removed joint left_wheel_joint
- removed joint right_wheel_joint
- added joint bot3_left_wheel_joint: type continuous, parent base_link, child left_wheel, origin xyz=-0.02 0.048  -0.015 rpy=0 1.570795 1.570795, axis 0 0 1
- added joint bot3_right_wheel_joint: type continuous, parent base_link, child right_wheel, origin xyz=-0.02 -0.048  -0.015 rpy=0 1.570795 1.570795, axis 0 0 1

File: software/bot_description/urdf/bot4.urdf (robot description, URDF)
Before this commit: robot bot4, 5 links, 4 joints
Links:
- link base_link_inertia: geometry collision box size=0.08 0.08 0.008; visual mesh filename=package://bot_description/meshes/bot4.dae scale=1.22 1.22 1.22
Joints:
- removed joint left_wheel_joint
- removed joint right_wheel_joint
- added joint bot4_left_wheel_joint: type continuous, parent base_link, child left_wheel, origin xyz=-0.02 0.048  -0.015 rpy=0 1.570795 1.570795, axis 0 0 1
- added joint bot4_right_wheel_joint: type continuous, parent base_link, child right_wheel, origin xyz=-0.02 -0.048  -0.015 rpy=0 1.570795 1.570795, axis 0 0 1

Commit message: height of camera is adjusted and factor retuned. add light in gazebo world for estimator.py to work properly

File: software/bot_description/urdf/arena.urdf (robot description, URDF)
Before this commit: robot arena1, 3 links, 2 joints
Joints:
- joint camera_joint: origin xyz=0 0 1.2 rpy=0 1.57079632679 0 -> xyz=0 0 1.65 rpy=0 1.57079632679 0
