Commit message: round2 ka arena and setup

File: software/bot_description/urdf/arena.urdf (robot description, URDF)
Before this commit: robot arena1, 3 links, 2 joints
Links:
- link arena: geometry collision box size=0.0001 0.0001 0.0001; visual mesh filename=package://bot_description/meshes/arena2.dae
Joints:
- joint world_arena: origin xyz=0 0 0.0001 rpy=0 0 0 -> xyz=0 0 0.0001 rpy=0 1.57 0

File: software/bot_description/urdf/bot.urdf (robot description, URDF)
Before this commit: robot bot, 5 links, 4 joints
Links:
- added link aruco, mass 0.1; collision mesh filename=package://bot_description/meshes/bot2.dae scale=1.25 1.25 1.25; visual mesh filename=package://bot_description/meshes/bot2.dae scale=1.25 1.25 1.25
- link base_link_inertia: geometry collision box size=0.08 0.08 0.008; visual box size=0.08 0.08 0.008
- link caster_wheel: mass 3 -> 4; geometry collision sphere radius=0.02; visual sphere radius=0.02
- link left_wheel: geometry collision cylinder length=0.008 radius=0.02; visual cylinder length=0.008 radius=0.02
- link right_wheel: geometry collision cylinder length=0.008 radius=0.02; visual cylinder length=0.008 radius=0.02
Joints:
- removed joint base_link_inertia_joint
- removed joint left_wheel_joint
- removed joint right_wheel_joint
- added joint aruco_joint_2: type fixed, parent base_link, child aruco, origin xyz=0 0 0.07 rpy=0 0 0
- added joint base_link_inertia_joint_2: type fixed, parent base_link, child base_link_inertia, origin xyz=0 0 0 rpy=0 0 0
- added joint bot2_left_wheel_joint: type continuous, parent base_link, child left_wheel, origin xyz=-0.03 0.048  -0.01 rpy=0 1.570795 1.570795, axis 0 0 1
- added joint bot2_right_wheel_joint: type continuous, parent base_link, child right_wheel, origin xyz=-0.03 -0.048  -0.01 rpy=0 1.570795 1.570795, axis 0 0 1
- joint caster_wheel_joint: origin xyz=0.04 0 -0.0491666666667 rpy=0 0 0 -> xyz=0.02 0 -0.01 rpy=0 0 0; type continuous -> fixed

File: software/bot_description/urdf/bot.urdf.xacro (robot description, xacro)
@@ -1,13 +1,13 @@
 <?xml version="1.0"?>
-<robot name="bot4" xmlns:xacro="http://ros.org/wiki/xacro">
-	<xacro:property name="wheel_dia" value="0.05"/>
-	<xacro:property name="bot_height" value="0.07"/>
+<robot name="bot1" xmlns:xacro="http://ros.org/wiki/xacro">
+	<xacro:property name="wheel_dia" value="0.04"/>
+	<xacro:property name="bot_height" value="0.03"/>
 	<xacro:property name="length" value="0.08"/>
 	<xacro:property name="breadth" value="0.08"/>
 	<xacro:property name="pi" value="3.14159"/>
 	<xacro:property name="m_base" value="1"/>
-	<xacro:property name="m_wheel" value="0.3"/>
-	<xacro:property name="m_aruco" value="0.1"/>
-	<xacro:property name="m_caster_wheel" value="4"/>
+	<xacro:property name="m_wheel" value="0.4"/>
+	<xacro:property name="m_aruco" value="0.04"/>
+	<xacro:property name="m_caster_wheel" value="0.1"/>
   	<xacro:property name="bot_number" value="1"/>
 	<link name="base_link"/>
@@ -25,9 +25,32 @@
 		</collision>
 		<visual>
-			<origin xyz="0 0 0.02" rpy="0 0 0"/>
+			<origin xyz="0 0 0" rpy="0 0 0"/>
 			<geometry>
 				<box size="${length} ${breadth} 0.008"/>
 			</geometry>
 		</visual>
+		<!-- caster -->
+	<!-- 	<collision name="caster_wheel_collision">
+			<origin xyz="${length/2-0.02} 0 -0.02" rpy="0 0 0"/>
+			<geometry>
+				<sphere radius="${wheel_dia/4.0}"/>
+			</geometry>
+			<surface>
+		        <friction>
+		          <ode>
+		            <mu>0</mu>
+		            <mu2>0</mu2>
+		            <slip1>1.0</slip1>
+		            <slip2>1.0</slip2>
+		          </ode>
+		        </friction>
+      		</surface>
+		</collision>
+		<visual name ="caster_wheel_visual">
+			<origin xyz="${length/2-0.02} 0 -0.02" rpy="0 0 0"/>
+			<geometry>
+				<sphere radius="${wheel_dia/4.0}"/>
+			</geometry>
+		</visual> -->
 	</link>
 	<link name="aruco">
@@ -88,38 +111,86 @@
 		</visual>
 	</link>
-	<link name="caster_wheel">
+	<link name="left_wheel_dumy">
+		<inertial>
+     		<origin xyz="0 0 0" rpy="0 0 0"/>
+     		<mass value="${m_wheel}"/>
+     		<inertia ixx="${m_wheel*(3*wheel_dia*wheel_dia/4.0+0.008*0.008)/12.0}"  ixy="0"  ixz="0" iyy="${m_wheel*(3*wheel_dia*wheel_dia/4.0+0.008*0.008)/12.0}" iyz="0" izz="${m_wheel*(wheel_dia*wheel_dia/4)/2.0}" />
+   		</inertial>
+		<collision>
+			<origin xyz="0 0 0" rpy="0 0 0"/>
+			<geometry>
+				<cylinder radius="${wheel_dia/2.0}" length="0.008"/>
+			</geometry>
+		</collision>
+		<visual>
+			<origin xyz="0 0 0" rpy="0 0 0"/>
+			<geometry>
+				<cylinder radius="${wheel_dia/2.0}" length="0.008"/>
+			</geometry>
+		</visual>
+	</link>
+	<link name="right_wheel_dumy">
+		<inertial>
+     		<origin xyz="0 0 0" rpy="0 0 0"/>
+     		<mass value="${m_wheel}"/>
+     		<inertia ixx="${m_wheel*(3*wheel_dia*wheel_dia/4.0+0.008*0.008)/12.0}"  ixy="0"  ixz="0" iyy="${m_wheel*(3*wheel_dia*wheel_dia/4.0+0.008*0.008)/12.0}" iyz="0" izz="${m_wheel*(wheel_dia*wheel_dia/4)/2.0}" />
+   		</inertial>
+		<collision>
+			<origin xyz="0 0 0" rpy="0 0 0"/>
+			<geometry>
+				<cylinder radius="${wheel_dia/2.0}" length="0.008"/>
+			</geometry>
+		</collision>
+		<visual>
+			<origin xyz="0 0 0" rpy="0 0 0"/>
+			<geometry>
+				<cylinder radius="${wheel_dia/2.0}" length="0.008"/>
+			</geometry>
+		</visual>
+	</link>
+	<!-- <link name="caster_wheel">
 		<inertial>
      		<origin xyz="0 0 0" rpy="0 0 0"/>
      		<mass value="${m_caster_wheel}"/>
-     		<inertia ixx="${m_caster_wheel*(2*wheel_dia*wheel_dia/9.0)/5.0}"  ixy="0"  ixz="0" iyy="${m_caster_wheel*(2*wheel_dia*wheel_dia/9.0)/5.0}" iyz="0" izz="${m_caster_wheel*(2*wheel_dia*wheel_dia/9.0)/5.0}" />
-   		</inertial>
-		<collision>
-			<origin xyz="0 0 0" rpy="0 0 0"/>
-			<geometry>
-				<sphere radius="${wheel_dia/3.0}"/>
-			</geometry>
-		</collision>
-		<visual>
-			<origin xyz="0 0 0" rpy="0 0 0"/>
-			<geometry>
-				<sphere radius="${wheel_dia/3.0}"/>
-			</geometry>
-		</visual>
-	</link>
+     		<inertia ixx="${m_caster_wheel*(2*wheel_dia*wheel_dia/16.0)/5.0}"  ixy="0"  ixz="0" iyy="${m_caster_wheel*(2*wheel_dia*wheel_dia/16.0)/5.0}" iyz="0" izz="${m_caster_wheel*(2*wheel_dia*wheel_dia/16.0)/5.0}" />
+   		</inertial>
+		<collision>
+			<origin xyz="0 0 0" rpy="0 0 0"/>
+			<geometry>
+				<sphere radius="${wheel_dia/4.0}"/>
+			</geometry>
+			<surface>
+		        <friction>
+		          <ode>
+		            <mu>0</mu>
+		            <mu2>0</mu2>
+		            <slip1>1.0</slip1>
+		            <slip2>1.0</slip2>
+		          </ode>
+		        </friction>
+      		</surface>
+		</collision>
+		<visual>
+			<origin xyz="0 0 0" rpy="0 0 0"/>
+			<geometry>
+				<sphere radius="${wheel_dia/4.0}"/>
+			</geometry>
+		</visual>
+	</link> -->
 <!-- joints def -->
-	<joint name="base_link_inertia_joint" type="fixed">
+	<joint name="base_link_inertia_joint_${bot_number}" type="fixed">
 		<parent link="base_link"/>
 		<child link="base_link_inertia"/>
 		<origin rpy="0 0 0" xyz="0 0 0"/>
 	</joint>
-	<joint name="aruco_joint" type="fixed">
+	<joint name="aruco_joint_${bot_number}" type="fixed">
 		<parent link="base_link"/>
 		<child link="aruco"/>
-		<origin rpy="0 0 0" xyz="0 0 0.05"/>
+		<origin rpy="0 0 0" xyz="0 0 0.07"/>
 	</joint>
 	<joint name="bot${bot_number}_left_wheel_joint" type="continuous">
 		<parent link="base_link"/>
 		<child link="left_wheel"/>
-		<origin rpy="0 ${pi/2} ${pi/2}" xyz="-0.02 ${breadth/2+0.008}  -0.015"/>
+		<origin rpy="0 ${pi/2} ${pi/2}" xyz="-0.03 ${breadth/2+0.008}  -0.01"/>
 		<axis rpy="0 0 0" xyz="0 0 1"/>
 	</joint>
@@ -127,39 +198,49 @@
 		<parent link="base_link"/>
 		<child link="right_wheel"/>
-		<origin rpy="0 ${pi/2} ${pi/2}" xyz="-0.02 ${-breadth/2-0.008}  -0.015"/>
-		<axis rpy="0 0 0" xyz="0 0 1"/>
-	</joint>
-	<joint name="caster_wheel_joint" type="continuous">
-		<parent link="base_link"/>
-		<child link="caster_wheel"/>
-		<origin rpy="0 0 0" xyz="${length/2-0.02} 0 ${-0.015- wheel_dia/6}"/>
-		<axis rpy="0 0 0" xyz="0 1 0"/>
+		<origin rpy="0 ${pi/2} ${pi/2}" xyz="-0.03 ${-breadth/2-0.008}  -0.01"/>
+		<axis rpy="0 0 0" xyz="0 0 1"/>
+	</joint>
+	<joint name="bot${bot_number}_left_wheel_joint_dumy" type="continuous">
+		<parent link="base_link"/>
+		<child link="left_wheel_dumy"/>
+		<origin rpy="0 ${pi/2} ${pi/2}" xyz="0.03 ${breadth/2+0.008}  -0.01"/>
+		<axis rpy="0 0 0" xyz="0 0 1"/>
+	</joint>
+	<joint name="bot${bot_number}_right_wheel_joint_dumy" type="continuous">
+		<parent link="base_link"/>
+		<child link="right_wheel_dumy"/>
+		<origin rpy="0 ${pi/2} ${pi/2}" xyz="0.03 ${-breadth/2-0.008}  -0.01"/>
+		<axis rpy="0 0 0" xyz="0 0 1"/>
 	</joint>
 	<!-- controls plugin for vlecoty based control -->
-	<gazebo>
-        <plugin name="gazebo_ros_control" filename="libgazebo_ros_control.so">
-            <legacyModeNS>true</legacyModeNS>
-            <robotNamespace>/bot${bot_number}</robotNamespace>
-        </plugin>
-	</gazebo>
-  <transmission name="bot${bot_number}_left_wheel_trans">
-    <type>transmission_interface/SimpleTransmission</type>
-    <joint name="bot${bot_number}_left_wheel_joint">
-        <hardwareInterface>hardware_interface/EffortJointInterface</hardwareInterface>
-    </joint>
-    <actuator name="bot${bot_number}_left_wheel_joint_motor">
-        <hardwareInterface>hardware_interface/EffortJointInterface</hardwareInterface>
-        <mechanicalReduction>1</mechanicalReduction>
-    </actuator>
-  </transmission>
-  <transmission name="bot${bot_number}_right_wheel_trans">
-    <type>transmission_interface/SimpleTransmission</type>
-    <joint name="bot${bot_number}_right_wheel_joint">
-        <hardwareInterface>hardware_interface/EffortJointInterface</hardwareInterface>
-    </joint>
-    <actuator name="bot${bot_number}_right_wheel_joint_motor">
-        <hardwareInterface>hardware_interface/EffortJointInterface</hardwareInterface>
-        <mechanicalReduction>1</mechanicalReduction>
-    </actuator>
-  </transmission>
+<gazebo>
+    <plugin filename="libgazebo_ros_diff_drive.so" name="differential_drive_controller">
+      <alwaysOn>true</alwaysOn>
+      <updateRate>2</updateRate>
+      <leftJoint>bot${bot_number}_left_wheel_joint</leftJoint>
+      <rightJoint>bot${bot_number}_right_wheel_joint</rightJoint>
+      <wheelSeparation>0.096</wheelSeparation>
+      <wheelDiameter>0.04</wheelDiameter>
+      <torque>1</torque>
+      <commandTopic>cmd_vel</commandTopic>
+      <odometryTopic>odom</odometryTopic>
+      <odometryFrame>odom</odometryFrame>
+      <robotBaseFrame>base_link</robotBaseFrame>
+    </plugin>
+  </gazebo>
+<gazebo>
+    <plugin filename="libgazebo_ros_diff_drive.so" name="differential_drive_controller">
+      <alwaysOn>true</alwaysOn>
+      <updateRate>2</updateRate>
+      <leftJoint>bot${bot_number}_left_wheel_joint_dumy</leftJoint>
+      <rightJoint>bot${bot_number}_right_wheel_joint_dumy</rightJoint>
+      <wheelSeparation>0.096</wheelSeparation>
+      <wheelDiameter>0.04</wheelDiameter>
+      <torque>1</torque>
+      <commandTopic>cmd_vel_dumy</commandTopic>
+      <odometryTopic>odom</odometryTopic>
+      <odometryFrame>odom</odometryFrame>
+      <robotBaseFrame>base_link</robotBaseFrame>
+    </plugin>
+  </gazebo>
 </robot>

File: software/bot_description/urdf/bot1.urdf (robot description, URDF)
Before this commit: robot bot1, 5 links, 4 joints
Links:
- removed link caster_wheel
- added link aruco, mass 0.04; collision mesh filename=package://bot_description/meshes/bot1.dae scale=1.25 1.25 1.25; visual mesh filename=package://bot_description/meshes/bot1.dae scale=1.25 1.25 1.25
- added link left_wheel_dumy, mass 0.4; collision cylinder length=0.008 radius=0.02; visual cylinder length=0.008 radius=0.02
- added link right_wheel_dumy, mass 0.4; collision cylinder length=0.008 radius=0.02; visual cylinder length=0.008 radius=0.02
- link base_link_inertia: geometry collision box size=0.08 0.08 0.008; visual box size=0.08 0.08 0.008
- link left_wheel: mass 0.3 -> 0.4; geometry collision cylinder length=0.008 radius=0.02; visual cylinder length=0.008 radius=0.02
- link right_wheel: mass 0.3 -> 0.4; geometry collision cylinder length=0.008 radius=0.02; visual cylinder length=0.008 radius=0.02
Joints:
- removed joint base_link_inertia_joint
- removed joint caster_wheel_joint
- added joint aruco_joint_1: type fixed, parent base_link, child aruco, origin xyz=0 0 0.07 rpy=0 0 0
- added joint base_link_inertia_joint_1: type fixed, parent base_link, child base_link_inertia, origin xyz=0 0 0 rpy=0 0 0
- added joint bot1_left_wheel_joint_dumy: type continuous, parent base_link, child left_wheel_dumy, origin xyz=0.03 0.048  -0.01 rpy=0 1.570795 1.570795, axis 0 0 1
- added joint bot1_right_wheel_joint_dumy: type continuous, parent base_link, child right_wheel_dumy, origin xyz=0.03 -0.048  -0.01 rpy=0 1.570795 1.570795, axis 0 0 1
- joint bot1_left_wheel_joint: origin xyz=-0.02 0.048  -0.015 rpy=0 1.570795 1.570795 -> xyz=-0.03 0.048  -0.01 rpy=0 1.570795 1.570795
- joint bot1_right_wheel_joint: origin xyz=-0.02 -0.048  -0.015 rpy=0 1.570795 1.570795 -> xyz=-0.03 -0.048  -0.01 rpy=0 1.570795 1.570795

File: software/bot_description/urdf/bot2.urdf (robot description, URDF)
Before this commit: robot bot2, 5 links, 4 joints
Links:
- removed link caster_wheel
- added link aruco, mass 0.04; collision mesh filename=package://bot_description/meshes/bot2.dae scale=1.25 1.25 1.25; visual mesh filename=package://bot_description/meshes/bot2.dae scale=1.25 1.25 1.25
- added link left_wheel_dumy, mass 0.4; collision cylinder length=0.008 radius=0.02; visual cylinder length=0.008 radius=0.02
- added link right_wheel_dumy, mass 0.4; collision cylinder length=0.008 radius=0.02; visual cylinder length=0.008 radius=0.02
- link base_link_inertia: geometry collision box size=0.08 0.08 0.008; visual box size=0.08 0.08 0.008
- link left_wheel: mass 0.3 -> 0.4; geometry collision cylinder length=0.008 radius=0.02; visual cylinder length=0.008 radius=0.02
- link right_wheel: mass 0.3 -> 0.4; geometry collision cylinder length=0.008 radius=0.02; visual cylinder length=0.008 radius=0.02
Joints:
- removed joint base_link_inertia_joint
- removed joint caster_wheel_joint
- added joint aruco_joint_2: type fixed, parent base_link, child aruco, origin xyz=0 0 0.07 rpy=0 0 0
- added joint base_link_inertia_joint_2: type fixed, parent base_link, child base_link_inertia, origin xyz=0 0 0 rpy=0 0 0
- added joint bot2_left_wheel_joint_dumy: type continuous, parent base_link, child left_wheel_dumy, origin xyz=0.03 0.048  -0.01 rpy=0 1.570795 1.570795, axis 0 0 1
- added joint bot2_right_wheel_joint_dumy: type continuous, parent base_link, child right_wheel_dumy, origin xyz=0.03 -0.048  -0.01 rpy=0 1.570795 1.570795, axis 0 0 1
- joint bot2_left_wheel_joint: origin xyz=-0.02 0.048  -0.015 rpy=0 1.570795 1.570795 -> xyz=-0.03 0.048  -0.01 rpy=0 1.570795 1.570795
- joint bot2_right_wheel_joint: origin xyz=-0.02 -0.048  -0.015 rpy=0 1.570795 1.570795 -> xyz=-0.03 -0.048  -0.01 rpy=0 1.570795 1.570795

File: software/bot_description/urdf/bot3.urdf (robot description, URDF)
Before this commit: robot bot3, 5 links, 4 joints
Links:
- removed link caster_wheel
- added link aruco, mass 0.04; collision mesh filename=package://bot_description/meshes/bot3.dae scale=1.25 1.25 1.25; visual mesh filename=package://bot_description/meshes/bot3.dae scale=1.25 1.25 1.25
- added link left_wheel_dumy, mass 0.4; collision cylinder length=0.008 radius=0.02; visual cylinder length=0.008 radius=0.02
- added link right_wheel_dumy, mass 0.4; collision cylinder length=0.008 radius=0.02; visual cylinder length=0.008 radius=0.02
- link base_link_inertia: geometry collision box size=0.08 0.08 0.008; visual box size=0.08 0.08 0.008
- link left_wheel: mass 0.3 -> 0.4; geometry collision cylinder length=0.008 radius=0.02; visual cylinder length=0.008 radius=0.02
- link right_wheel: mass 0.3 -> 0.4; geometry collision cylinder length=0.008 radius=0.02; visual cylinder length=0.008 radius=0.02
Joints:
- removed joint base_link_inertia_joint
- removed joint caster_wheel_joint
- added joint aruco_joint_3: type fixed, parent base_link, child aruco, origin xyz=0 0 0.07 rpy=0 0 0
- added joint base_link_inertia_joint_3: type fixed, parent base_link, child base_link_inertia, origin xyz=0 0 0 rpy=0 0 0
- added joint bot3_left_wheel_joint_dumy: type continuous, parent base_link, child left_wheel_dumy, origin xyz=0.03 0.048  -0.01 rpy=0 1.570795 1.570795, axis 0 0 1
- added joint bot3_right_wheel_joint_dumy: type continuous, parent base_link, child right_wheel_dumy, origin xyz=0.03 -0.048  -0.01 rpy=0 1.570795 1.570795, axis 0 0 1
- joint bot3_left_wheel_joint: origin xyz=-0.02 0.048  -0.015 rpy=0 1.570795 1.570795 -> xyz=-0.03 0.048  -0.01 rpy=0 1.570795 1.570795
- joint bot3_right_wheel_joint: origin xyz=-0.02 -0.048  -0.015 rpy=0 1.570795 1.570795 -> xyz=-0.03 -0.048  -0.01 rpy=0 1.570795 1.570795

File: software/bot_description/urdf/bot4.urdf (robot description, URDF)
Before this commit: robot bot4, 5 links, 4 joints
Links:
- removed link caster_wheel
- added link aruco, mass 0.04; collision mesh filename=package://bot_description/meshes/bot4.dae scale=1.25 1.25 1.25; visual mesh filename=package://bot_description/meshes/bot4.dae scale=1.25 1.25 1.25
- added link left_wheel_dumy, mass 0.4; collision cylinder length=0.008 radius=0.02; visual cylinder length=0.008 radius=0.02
- added link right_wheel_dumy, mass 0.4; collision cylinder length=0.008 radius=0.02; visual cylinder length=0.008 radius=0.02
- link base_link_inertia: geometry collision box size=0.08 0.08 0.008; visual box size=0.08 0.08 0.008
- link left_wheel: mass 0.3 -> 0.4; geometry collision cylinder length=0.008 radius=0.02; visual cylinder length=0.008 radius=0.02
- link right_wheel: mass 0.3 -> 0.4; geometry collision cylinder length=0.008 radius=0.02; visual cylinder length=0.008 radius=0.02
Joints:
- removed joint base_link_inertia_joint
- removed joint caster_wheel_joint
- added joint aruco_joint_4: type fixed, parent base_link, child aruco, origin xyz=0 0 0.07 rpy=0 0 0
- added joint base_link_inertia_joint_4: type fixed, parent base_link, child base_link_inertia, origin xyz=0 0 0 rpy=0 0 0
- added joint bot4_left_wheel_joint_dumy: type continuous, parent base_link, child left_wheel_dumy, origin xyz=0.03 0.048  -0.01 rpy=0 1.570795 1.570795, axis 0 0 1
- added joint bot4_right_wheel_joint_dumy: type continuous, parent base_link, child right_wheel_dumy, origin xyz=0.03 -0.048  -0.01 rpy=0 1.570795 1.570795, axis 0 0 1
- joint bot4_left_wheel_joint: origin xyz=-0.02 0.048  -0.015 rpy=0 1.570795 1.570795 -> xyz=-0.03 0.048  -0.01 rpy=0 1.570795 1.570795
- joint bot4_right_wheel_joint: origin xyz=-0.02 -0.048  -0.015 rpy=0 1.570795 1.570795 -> xyz=-0.03 -0.048  -0.01 rpy=0 1.570795 1.570795

Commit message: cbs code has been added and it has been interfacted with ROS. topic /start_goal_agent for input and /cbs/plan for output

File: software/bot_description/urdf/arena.urdf (robot description, URDF)
Before this commit: robot arena2, 3 links, 2 joints
Joints:
- joint world_arena: origin xyz=0 0 0.0001 rpy=0 1.57 0 -> xyz=0 0 0.0001 rpy=0 0 0

Commit message: pid needs tuning

File: software/bot_description/urdf/arena.urdf (robot description, URDF)
Before this commit: robot arena2, 3 links, 2 joints
Joints:
- joint world_arena: origin xyz=0 0 0.0001 rpy=0 0 0 -> xyz=0 0 0.0001 rpy=0 0 1.57079

File: software/bot_description/urdf/bot.urdf.xacro (robot description, xacro)
@@ -1,4 +1,4 @@
 <?xml version="1.0"?>
-<robot name="bot3" xmlns:xacro="http://ros.org/wiki/xacro">
+<robot name="bot0" xmlns:xacro="http://ros.org/wiki/xacro">
 	<xacro:property name="wheel_dia" value="0.04"/>
 	<xacro:property name="bot_height" value="0.03"/>
@@ -10,5 +10,5 @@
 	<xacro:property name="m_aruco" value="0.04"/>
 	<xacro:property name="m_caster_wheel" value="0.1"/>
-  	<xacro:property name="bot_number" value="3"/>
+  	<xacro:property name="bot_number" value="0"/>
 	<link name="base_link"/>
 	<link name="base_link_inertia">
@@ -63,11 +63,11 @@
 			<origin xyz="0 0 0" rpy="0 0 0"/>
 			<geometry>
-				 <mesh filename="package://bot_description/meshes/bot${bot_number}.dae" scale="1.25 1.25 1.25"/>
-			</geometry>
-		</collision>
-		<visual>
-			<origin xyz="0 0 0" rpy="0 0 0"/>
-			<geometry>
-				 <mesh filename="package://bot_description/meshes/bot${bot_number}.dae" scale="1.25 1.25 1.25"/>
+				 <mesh filename="package://bot_description/meshes/bot${bot_number+1}.dae" scale="1.25 1.25 1.25"/>
+			</geometry>
+		</collision>
+		<visual>
+			<origin xyz="0 0 0" rpy="0 0 0"/>
+			<geometry>
+				 <mesh filename="package://bot_description/meshes/bot${bot_number+1}.dae" scale="1.25 1.25 1.25"/>
 			</geometry>
 		</visual>

File: software/bot_description/urdf/bot1.urdf (robot description, URDF)
Before this commit: robot bot0, 7 links, 6 joints
Links:
- link aruco: geometry collision mesh filename=package://bot_description/meshes/bot1.dae scale=1.25 1.25 1.25; visual mesh filename=package://bot_description/meshes/bot1.dae scale=1.25 1.25 1.25

File: software/bot_description/urdf/bot2.urdf (robot description, URDF)
Before this commit: robot bot1, 7 links, 6 joints
Links:
- link aruco: geometry collision mesh filename=package://bot_description/meshes/bot2.dae scale=1.25 1.25 1.25; visual mesh filename=package://bot_description/meshes/bot2.dae scale=1.25 1.25 1.25

File: software/bot_description/urdf/bot3.urdf (robot description, URDF)
Before this commit: robot bot2, 7 links, 6 joints
Links:
- link aruco: geometry collision mesh filename=package://bot_description/meshes/bot3.dae scale=1.25 1.25 1.25; visual mesh filename=package://bot_description/meshes/bot3.dae scale=1.25 1.25 1.25

File: software/bot_description/urdf/bot4.urdf (robot description, URDF)
Before this commit: robot bot3, 7 links, 6 joints
Links:
- link aruco: geometry collision mesh filename=package://bot_description/meshes/bot4.dae scale=1.25 1.25 1.25; visual mesh filename=package://bot_description/meshes/bot4.dae scale=1.25 1.25 1.25
