Commit message: changes commited for nitish reference

File: software/bot_description/urdf/arena.urdf (robot description, URDF)
Before this commit: robot arena2, 3 links, 2 joints
Links:
- added link wall1_x, mass 1; collision box size=0.01 2.1336 0.0254; visual box size=0.01 2.1336 0.0254
- added link wall1_x1, mass 1; collision box size=0.01 0.3048 0.0254; collision box size=0.01 0.3048 0.0254
- added link wall1_y, mass 1; collision box size=2.1336 0.01 0.0254; visual box size=2.1336 0.01 0.0254
- added link wall1_y1, mass 1; collision box size=0.3048 0.001 0.0254; collision box size=0.3048 0.001 0.0254
- added link wall2_x, mass 1; collision box size=0.01 2.1336 0.0254; visual box size=0.01 2.1336 0.0254
- added link wall2_x1, mass 1; collision box size=0.01 0.3048 0.0254; collision box size=0.01 0.3048 0.0254
- added link wall2_y, mass 1; collision box size=2.1336 0.01 0.0254; visual box size=2.1336 0.01 0.0254
- added link wall2_y1, mass 1; collision box size=0.3048 0.001 0.0254; collision box size=0.3048 0.001 0.0254
Joints:
- added joint wal2_x1_joint: type fixed, parent world, child wall2_x1, origin xyz=-0.1524 0 0.0127 rpy=0 0 0, axis 0 1 0
- added joint wal2_x_joint: type fixed, parent world, child wall2_x, origin xyz=-1.0668 0 0.0127 rpy=0 0 0, axis 0 1 0
- added joint wall1_x1_joint: type fixed, parent world, child wall1_x1, origin xyz=0.1524 0 0.0127 rpy=0 0 0, axis 0 1 0
- added joint wall1_x_joint: type fixed, parent world, child wall1_x, origin xyz=1.0668 0 0.0127 rpy=0 0 0, axis 0 1 0
- added joint wall1_y1_joint: type fixed, parent world, child wall1_y1, origin xyz=0 0.1524 0.0127 rpy=0 0 0, axis 0 1 0
- added joint wall1_y_joint: type fixed, parent world, child wall1_y, origin xyz=0 1.0668 0.0127 rpy=0 0 0, axis 0 1 0
- added joint wall2_y1_joint: type fixed, parent world, child wall2_y1, origin xyz=0 -0.1524 0.0127 rpy=0 0 0, axis 0 1 0
- added joint wall2_y_joint: type fixed, parent world, child wall2_y, origin xyz=0 -1.0668 0.0127 rpy=0 0 0, axis 0 1 0
