Commit message: on going work on individual control of each wheel

File: software/bot_description/urdf/bot.urdf.xacro (robot description, xacro)
@@ -1,5 +1,4 @@
 <?xml version="1.0"?>
-<robot name="bot" xmlns:xacro="http://ros.org/wiki/xacro">
-	<!-- <xacro:include filename="$(find bot_description)/urdf/" /> -->
+<robot name="bot1" xmlns:xacro="http://ros.org/wiki/xacro">
 	<xacro:property name="wheel_dia" value="0.05"/>
 	<xacro:property name="bot_height" value="0.07"/>
@@ -10,4 +9,5 @@
 	<xacro:property name="m_wheel" value="0.3"/>
 	<xacro:property name="m_caster_wheel" value="3"/>
+  <xacro:property name="bot_number" value="1"/>
 	<link name="base_link"/>
 	<link name="base_link_inertia">
@@ -26,5 +26,5 @@
 			<origin xyz="0 0 0" rpy="0 0 0"/>
 			<geometry>
-				<mesh filename="package://bot_description/meshes/bot1.dae"  />
+				<mesh filename="package://bot_description/meshes/bot${bot_number}.dae"  />
 			</geometry>
 		</visual>
@@ -87,4 +87,5 @@
 		</visual>
 	</link>
+<!-- joints def -->
 	<joint name="base_link_inertia_joint" type="fixed">
 		<parent link="base_link"/>
@@ -92,5 +93,5 @@
 		<origin rpy="0 0 0" xyz="0 0 0"/>
 	</joint>
-	<joint name="left_wheel_joint" type="continuous">
+	<joint name="bot${bot_number}_left_wheel_joint" type="continuous">
 		<parent link="base_link"/>
 		<child link="left_wheel"/>
@@ -98,5 +99,5 @@
 		<axis rpy="0 0 0" xyz="0 0 1"/>
 	</joint>
-	<joint name="right_wheel_joint" type="continuous">
+	<joint name="bot${bot_number}_right_wheel_joint" type="continuous">
 		<parent link="base_link"/>
 		<child link="right_wheel"/>
@@ -110,18 +111,30 @@
 		<axis rpy="0 0 0" xyz="0 1 0"/>
 	</joint>
+	<!-- controls plugin for vlecoty based control -->
 	<gazebo>
-    <plugin filename="libgazebo_ros_diff_drive.so" name="differential_drive_controller">
-      <alwaysOn>true</alwaysOn>
-      <updateRate>20</updateRate>
-      <leftJoint>left_wheel_joint</leftJoint>
-      <rightJoint>right_wheel_joint</rightJoint>
-      <wheelSeparation>${breadth+0.016}</wheelSeparation>
-      <wheelDiameter>${wheel_dia}</wheelDiameter>
-      <torque>0.001</torque>
-      <commandTopic>cmd_vel</commandTopic>
-      <odometryTopic>odom</odometryTopic>
-      <odometryFrame>odom</odometryFrame>
-      <robotBaseFrame>base_link</robotBaseFrame>
-    </plugin>
-  </gazebo>
+        <plugin name="gazebo_ros_control" filename="libgazebo_ros_control.so">
+            <legacyModeNS>true</legacyModeNS>
+            <robotNamespace>/bot${bot_number}</robotNamespace>
+        </plugin>
+	</gazebo>
+  <transmission name="bot${bot_number}_left_wheel_trans">
+    <type>transmission_interface/SimpleTransmission</type>
+    <joint name="bot${bot_number}_left_wheel_joint">
+        <hardwareInterface>hardware_interface/EffortJointInterface</hardwareInterface>
+    </joint>
+    <actuator name="bot${bot_number}_left_wheel_joint_motor">
+        <hardwareInterface>hardware_interface/EffortJointInterface</hardwareInterface>
+        <mechanicalReduction>1</mechanicalReduction>
+    </actuator>
+  </transmission>
+  <transmission name="bot${bot_number}_right_wheel_trans">
+    <type>transmission_interface/SimpleTransmission</type>
+    <joint name="bot${bot_number}_right_wheel_joint">
+        <hardwareInterface>hardware_interface/EffortJointInterface</hardwareInterface>
+    </joint>
+    <actuator name="bot${bot_number}_right_wheel_joint_motor">
+        <hardwareInterface>hardware_interface/EffortJointInterface</hardwareInterface>
+        <mechanicalReduction>1</mechanicalReduction>
+    </actuator>
+  </transmission>
 </robot>

Commit message: height of camera is adjusted and factor retuned. add light in gazebo world for estimator.py to work properly

File: software/bot_description/urdf/bot.urdf.xacro (robot description, xacro)
@@ -1,4 +1,4 @@
 <?xml version="1.0"?>
-<robot name="bot1" xmlns:xacro="http://ros.org/wiki/xacro">
+<robot name="bot4" xmlns:xacro="http://ros.org/wiki/xacro">
 	<xacro:property name="wheel_dia" value="0.05"/>
 	<xacro:property name="bot_height" value="0.07"/>
@@ -8,5 +8,6 @@
 	<xacro:property name="m_base" value="1"/>
 	<xacro:property name="m_wheel" value="0.3"/>
-	<xacro:property name="m_caster_wheel" value="3"/>
+	<xacro:property name="m_aruco" value="0.1"/>
+	<xacro:property name="m_caster_wheel" value="4"/>
   <xacro:property name="bot_number" value="1"/>
 	<link name="base_link"/>
@@ -26,5 +27,24 @@
 			<origin xyz="0 0 0" rpy="0 0 0"/>
 			<geometry>
-				<mesh filename="package://bot_description/meshes/bot${bot_number}.dae"  />
+				<box size="${length} ${breadth} 0.008"/>
+			</geometry>
+		</visual>
+	</link>
+	<link name="aruco">
+		<inertial>
+     		<origin xyz="0 0 0" rpy="0 0 0"/>
+     		<mass value="${m_aruco}"/>
+     		<inertia ixx="${m_aruco*(breadth*breadth+0.008*0.008)/12.0}"  ixy="0"  ixz="0" iyy="${m_aruco*(length*length+0.008*0.008)/12.0}" iyz="0" izz="${m_aruco*(breadth*breadth+length*length)/12.0}" />
+   		</inertial>
+		<collision>
+			<origin xyz="0 0 0" rpy="0 0 0"/>
+			<geometry>
+				 <mesh filename="package://bot_description/meshes/bot${bot_number}.dae" scale="1.25 1.25 1.25"/>
+			</geometry>
+		</collision>
+		<visual>
+			<origin xyz="0 0 0" rpy="0 0 0"/>
+			<geometry>
+				 <mesh filename="package://bot_description/meshes/bot${bot_number}.dae" scale="1.25 1.25 1.25"/>
 			</geometry>
 		</visual>
@@ -93,4 +113,9 @@
 		<origin rpy="0 0 0" xyz="0 0 0"/>
 	</joint>
+	<joint name="aruco_joint" type="fixed">
+		<parent link="base_link"/>
+		<child link="aruco"/>
+		<origin rpy="0 0 0" xyz="0 0 0.05"/>
+	</joint>
 	<joint name="bot${bot_number}_left_wheel_joint" type="continuous">
 		<parent link="base_link"/>

Commit message: all 4 code working. need to make somemore changes

File: software/bot_description/urdf/bot.urdf.xacro (robot description, xacro)
@@ -1,4 +1,4 @@
 <?xml version="1.0"?>
-<robot name="bot1" xmlns:xacro="http://ros.org/wiki/xacro">
+<robot name="bot3" xmlns:xacro="http://ros.org/wiki/xacro">
 	<xacro:property name="wheel_dia" value="0.04"/>
 	<xacro:property name="bot_height" value="0.03"/>
@@ -10,5 +10,5 @@
 	<xacro:property name="m_aruco" value="0.04"/>
 	<xacro:property name="m_caster_wheel" value="0.1"/>
-  	<xacro:property name="bot_number" value="1"/>
+  	<xacro:property name="bot_number" value="3"/>
 	<link name="base_link"/>
 	<link name="base_link_inertia">

File: software/bot_description/urdf/bot1.urdf (robot description, URDF)
Before this commit: robot bot1, 7 links, 6 joints
Links:
- link aruco: geometry collision mesh filename=package://bot_description/meshes/bot0.dae scale=1.25 1.25 1.25; visual mesh filename=package://bot_description/meshes/bot0.dae scale=1.25 1.25 1.25
Joints:
- removed joint aruco_joint_1
- removed joint base_link_inertia_joint_1
- removed joint bot1_left_wheel_joint
- removed joint bot1_left_wheel_joint_dumy
- removed joint bot1_right_wheel_joint
- removed joint bot1_right_wheel_joint_dumy
- added joint aruco_joint_0: type fixed, parent base_link, child aruco, origin xyz=0 0 0.07 rpy=0 0 0
- added joint base_link_inertia_joint_0: type fixed, parent base_link, child base_link_inertia, origin xyz=0 0 0 rpy=0 0 0
- added joint bot0_left_wheel_joint: type continuous, parent base_link, child left_wheel, origin xyz=-0.03 0.048  -0.01 rpy=0 1.570795 1.570795, axis 0 0 1
- added joint bot0_left_wheel_joint_dumy: type continuous, parent base_link, child left_wheel_dumy, origin xyz=0.03 0.048  -0.01 rpy=0 1.570795 1.570795, axis 0 0 1
- added joint bot0_right_wheel_joint: type continuous, parent base_link, child right_wheel, origin xyz=-0.03 -0.048  -0.01 rpy=0 1.570795 1.570795, axis 0 0 1
- added joint bot0_right_wheel_joint_dumy: type continuous, parent base_link, child right_wheel_dumy, origin xyz=0.03 -0.048  -0.01 rpy=0 1.570795 1.570795, axis 0 0 1

File: software/bot_description/urdf/bot2.urdf (robot description, URDF)
Before this commit: robot bot2, 7 links, 6 joints
Links:
- link aruco: geometry collision mesh filename=package://bot_description/meshes/bot1.dae scale=1.25 1.25 1.25; visual mesh filename=package://bot_description/meshes/bot1.dae scale=1.25 1.25 1.25
Joints:
- removed joint aruco_joint_2
- removed joint base_link_inertia_joint_2
- removed joint bot2_left_wheel_joint
- removed joint bot2_left_wheel_joint_dumy
- removed joint bot2_right_wheel_joint
- removed joint bot2_right_wheel_joint_dumy
- added joint aruco_joint_1: type fixed, parent base_link, child aruco, origin xyz=0 0 0.07 rpy=0 0 0
- added joint base_link_inertia_joint_1: type fixed, parent base_link, child base_link_inertia, origin xyz=0 0 0 rpy=0 0 0
- added joint bot1_left_wheel_joint: type continuous, parent base_link, child left_wheel, origin xyz=-0.03 0.048  -0.01 rpy=0 1.570795 1.570795, axis 0 0 1
- added joint bot1_left_wheel_joint_dumy: type continuous, parent base_link, child left_wheel_dumy, origin xyz=0.03 0.048  -0.01 rpy=0 1.570795 1.570795, axis 0 0 1
- added joint bot1_right_wheel_joint: type continuous, parent base_link, child right_wheel, origin xyz=-0.03 -0.048  -0.01 rpy=0 1.570795 1.570795, axis 0 0 1
- added joint bot1_right_wheel_joint_dumy: type continuous, parent base_link, child right_wheel_dumy, origin xyz=0.03 -0.048  -0.01 rpy=0 1.570795 1.570795, axis 0 0 1

File: software/bot_description/urdf/bot3.urdf (robot description, URDF)
Before this commit: robot bot3, 7 links, 6 joints
Links:
- link aruco: geometry collision mesh filename=package://bot_description/meshes/bot2.dae scale=1.25 1.25 1.25; visual mesh filename=package://bot_description/meshes/bot2.dae scale=1.25 1.25 1.25
Joints:
- removed joint aruco_joint_3
- removed joint base_link_inertia_joint_3
- removed joint bot3_left_wheel_joint
- removed joint bot3_left_wheel_joint_dumy
- removed joint bot3_right_wheel_joint
- removed joint bot3_right_wheel_joint_dumy
- added joint aruco_joint_2: type fixed, parent base_link, child aruco, origin xyz=0 0 0.07 rpy=0 0 0
- added joint base_link_inertia_joint_2: type fixed, parent base_link, child base_link_inertia, origin xyz=0 0 0 rpy=0 0 0
- added joint bot2_left_wheel_joint: type continuous, parent base_link, child left_wheel, origin xyz=-0.03 0.048  -0.01 rpy=0 1.570795 1.570795, axis 0 0 1
- added joint bot2_left_wheel_joint_dumy: type continuous, parent base_link, child left_wheel_dumy, origin xyz=0.03 0.048  -0.01 rpy=0 1.570795 1.570795, axis 0 0 1
- added joint bot2_right_wheel_joint: type continuous, parent base_link, child right_wheel, origin xyz=-0.03 -0.048  -0.01 rpy=0 1.570795 1.570795, axis 0 0 1
- added joint bot2_right_wheel_joint_dumy: type continuous, parent base_link, child right_wheel_dumy, origin xyz=0.03 -0.048  -0.01 rpy=0 1.570795 1.570795, axis 0 0 1

File: software/bot_description/urdf/bot4.urdf (robot description, URDF)
Before this commit: robot bot4, 7 links, 6 joints
Links:
- link aruco: geometry collision mesh filename=package://bot_description/meshes/bot3.dae scale=1.25 1.25 1.25; visual mesh filename=package://bot_description/meshes/bot3.dae scale=1.25 1.25 1.25
Joints:
- removed joint aruco_joint_4
- removed joint base_link_inertia_joint_4
- removed joint bot4_left_wheel_joint
- removed joint bot4_left_wheel_joint_dumy
- removed joint bot4_right_wheel_joint
- removed joint bot4_right_wheel_joint_dumy
- added joint aruco_joint_3: type fixed, parent base_link, child aruco, origin xyz=0 0 0.07 rpy=0 0 0
- added joint base_link_inertia_joint_3: type fixed, parent base_link, child base_link_inertia, origin xyz=0 0 0 rpy=0 0 0
- added joint bot3_left_wheel_joint: type continuous, parent base_link, child left_wheel, origin xyz=-0.03 0.048  -0.01 rpy=0 1.570795 1.570795, axis 0 0 1
- added joint bot3_left_wheel_joint_dumy: type continuous, parent base_link, child left_wheel_dumy, origin xyz=0.03 0.048  -0.01 rpy=0 1.570795 1.570795, axis 0 0 1
- added joint bot3_right_wheel_joint: type continuous, parent base_link, child right_wheel, origin xyz=-0.03 -0.048  -0.01 rpy=0 1.570795 1.570795, axis 0 0 1
- added joint bot3_right_wheel_joint_dumy: type continuous, parent base_link, child right_wheel_dumy, origin xyz=0.03 -0.048  -0.01 rpy=0 1.570795 1.570795, axis 0 0 1

Commit message: mving from gazebo to matla for testing algo

File: software/bot_description/urdf/bot.urdf.xacro (robot description, xacro)
@@ -4,7 +4,10 @@
 	<xacro:property name="bot_height" value="0.03"/>
 	<xacro:property name="length" value="0.08"/>
-	<xacro:property name="breadth" value="0.08"/>
+	<xacro:property name="breadth" value="0.1"/>
+	<xacro:property name="length_" value="0.05"/>
+	<xacro:property name="breadth_" value="0.005"/>
 	<xacro:property name="pi" value="3.14159"/>
 	<xacro:property name="m_base" value="1"/>
+	<xacro:property name="m_lever" value="0.1"/>
 	<xacro:property name="m_wheel" value="0.4"/>
 	<xacro:property name="m_aruco" value="0.04"/>
@@ -73,4 +76,5 @@
 		</visual>
 	</link>
+<!-- x  direction wheel -->
 	<link name="left_wheel">
 		<inertial>
@@ -149,33 +153,24 @@
 		</visual>
 	</link>
-	<!-- <link name="caster_wheel">
-		<inertial>
-     		<origin xyz="0 0 0" rpy="0 0 0"/>
-     		<mass value="${m_caster_wheel}"/>
-     		<inertia ixx="${m_caster_wheel*(2*wheel_dia*wheel_dia/16.0)/5.0}"  ixy="0"  ixz="0" iyy="${m_caster_wheel*(2*wheel_dia*wheel_dia/16.0)/5.0}" iyz="0" izz="${m_caster_wheel*(2*wheel_dia*wheel_dia/16.0)/5.0}" />
-   		</inertial>
-		<collision>
-			<origin xyz="0 0 0" rpy="0 0 0"/>
-			<geometry>
-				<sphere radius="${wheel_dia/4.0}"/>
-			</geometry>
-			<surface>
-		        <friction>
-		          <ode>
-		            <mu>0</mu>
-		            <mu2>0</mu2>
-		            <slip1>1.0</slip1>
-		            <slip2>1.0</slip2>
-		          </ode>
-		        </friction>
-      		</surface>
-		</collision>
-		<visual>
-			<origin xyz="0 0 0" rpy="0 0 0"/>
-			<geometry>
-				<sphere radius="${wheel_dia/4.0}"/>
-			</geometry>
-		</visual>
-	</link> -->
+<!-- y direction wheel -->
+	<link name="back_right_wheel_lever">
+		<inertial>
+     		<origin xyz="0 0 0" rpy="0 0 0"/>
+     		<mass value="${m_lever}"/>
+     		<inertia ixx="${m_lever*(breadth_*breadth_+0.008*0.008)/12.0}"  ixy="0"  ixz="0" iyy="${m_lever*(length_*length_+0.008*0.008)/12.0}" iyz="0" izz="${m_lever*(breadth_*breadth_+length_*length_)/12.0}" />
+   		</inertial>
+		<collision>
+			<origin xyz="0 0.02 0" rpy="0 0 0"/>
+			<geometry>
+				<box size="0.008 ${length_} ${breadth_}"/>
+			</geometry>
+		</collision>
+		<visual>
+			<origin xyz="0 0.02 0" rpy="0 0 0"/>
+			<geometry>
+				<box size="0.008 ${length_} ${breadth_}"/>
+			</geometry>
+		</visual>
+	</link>
 <!-- joints def -->
 	<joint name="base_link_inertia_joint_${bot_number}" type="fixed">
@@ -192,5 +187,5 @@
 		<parent link="base_link"/>
 		<child link="left_wheel"/>
-		<origin rpy="0 ${pi/2} ${pi/2}" xyz="-0.03 ${breadth/2+0.008}  -0.01"/>
+		<origin rpy="0 ${pi/2} ${pi/2}" xyz="-0.022 ${breadth/2+0.006}  -0.01"/>
 		<axis rpy="0 0 0" xyz="0 0 1"/>
 	</joint>
@@ -198,5 +193,5 @@
 		<parent link="base_link"/>
 		<child link="right_wheel"/>
-		<origin rpy="0 ${pi/2} ${pi/2}" xyz="-0.03 ${-breadth/2-0.008}  -0.01"/>
+		<origin rpy="0 ${pi/2} ${pi/2}" xyz="-0.022 ${-breadth/2-0.006}  -0.01"/>
 		<axis rpy="0 0 0" xyz="0 0 1"/>
 	</joint>
@@ -204,5 +199,5 @@
 		<parent link="base_link"/>
 		<child link="left_wheel_dumy"/>
-		<origin rpy="0 ${pi/2} ${pi/2}" xyz="0.03 ${breadth/2+0.008}  -0.01"/>
+		<origin rpy="0 ${pi/2} ${pi/2}" xyz="0.022 ${breadth/2+0.006}  -0.01"/>
 		<axis rpy="0 0 0" xyz="0 0 1"/>
 	</joint>
@@ -210,6 +205,13 @@
 		<parent link="base_link"/>
 		<child link="right_wheel_dumy"/>
-		<origin rpy="0 ${pi/2} ${pi/2}" xyz="0.03 ${-breadth/2-0.008}  -0.01"/>
-		<axis rpy="0 0 0" xyz="0 0 1"/>
+		<origin rpy="0 ${pi/2} ${pi/2}" xyz="0.022 ${-breadth/2-0.006}  -0.01"/>
+		<axis rpy="0 0 0" xyz="0 0 1"/>
+	</joint>
+<!-- y direction level joints -->
+	<joint name="bot${bot_number}_back_right_wheel_lever" type="continuous">
+		<parent link="base_link"/>
+		<child link="back_right_wheel_lever"/>
+		<origin rpy="0 0 0" xyz="${-length/2-0.006} -0.04  -0.005"/>
+		<axis rpy="0 0 0" xyz="1 0 0"/>
 	</joint>
 	<!-- controls plugin for vlecoty based control -->
@@ -223,5 +225,5 @@
       <wheelDiameter>0.04</wheelDiameter>
       <torque>1</torque>
-      <commandTopic>cmd_vel</commandTopic>
+      <commandTopic>cmd_vel_x</commandTopic>
       <odometryTopic>odom</odometryTopic>
       <odometryFrame>odom</odometryFrame>
@@ -238,5 +240,5 @@
       <wheelDiameter>0.04</wheelDiameter>
       <torque>1</torque>
-      <commandTopic>cmd_vel_dumy</commandTopic>
+      <commandTopic>cmd_vel_dumy_x</commandTopic>
       <odometryTopic>odom</odometryTopic>
       <odometryFrame>odom</odometryFrame>

File: software/bot_description/urdf/bot1.urdf (robot description, URDF)
Before this commit: robot bot0, 7 links, 6 joints
Links:
- added link back_right_wheel_lever, mass 0.1; collision box size=0.008 0.05 0.005; visual box size=0.008 0.05 0.005
- link base_link_inertia: geometry collision box size=0.08 0.1 0.008; visual box size=0.08 0.1 0.008
Joints:
- added joint bot0_back_right_wheel_lever: type continuous, parent base_link, child back_right_wheel_lever, origin xyz=-0.046 -0.04  -0.005 rpy=0 0 0, axis 1 0 0
- joint bot0_left_wheel_joint: origin xyz=-0.03 0.048  -0.01 rpy=0 1.570795 1.570795 -> xyz=-0.022 0.056  -0.01 rpy=0 1.570795 1.570795
- joint bot0_left_wheel_joint_dumy: origin xyz=0.03 0.048  -0.01 rpy=0 1.570795 1.570795 -> xyz=0.022 0.056  -0.01 rpy=0 1.570795 1.570795
- joint bot0_right_wheel_joint: origin xyz=-0.03 -0.048  -0.01 rpy=0 1.570795 1.570795 -> xyz=-0.022 -0.056  -0.01 rpy=0 1.570795 1.570795
- joint bot0_right_wheel_joint_dumy: origin xyz=0.03 -0.048  -0.01 rpy=0 1.570795 1.570795 -> xyz=0.022 -0.056  -0.01 rpy=0 1.570795 1.570795
